Commit message: read me, docs

File: erl_assignment3/urdf/sherlock_robot.xacro (robot description, xacro)
@@ -167,5 +167,5 @@
   <joint name="camera_joint" type="fixed">
 	    <axis xyz="0 1 0" />
-	    <origin xyz="0.6 0 0.5" rpy="0 0 0"/>
+	    <origin xyz="0.3 0 0.5" rpy="0 0 0"/>
 	    <parent link="link_chassis"/>
 	    <child link="camera_link"/>
@@ -195,5 +195,5 @@
   <joint name="camera_floor_joint" type="fixed">
 	    <axis xyz="0 1 0" />
-	    <origin xyz="0.8 0 0.8" rpy="0 1.57 0"/>
+	    <origin xyz="0.5 0 0.5" rpy="0 1.57 0"/>
 	    <parent link="link_chassis"/>
 	    <child link="camera_floor_link"/>
